File: codemyriad-protogon.kicad_sch (KiCad schematic)
At the start: 13 parts, among them J1 Hexpansion-Connector, J2 Conn_02x10_Odd_Even, P1 PZ254V-11-02P, U1 ZD24C64A-XGMT, U2 SM04B-SRSS-TB_(LF)(SN)

Commit message: Rework the P1 jumper so it write-protects the EEPROM
P1 pin 2 now goes to +3V3 instead of GND, so shorting the jumper pulls WP
high and write-protects the EEPROM after provisioning. R3 still pulls WP low,
so the part is writable by default for the badge to provision. Board files
from the designer's reworked version.

- Update .kicad_pcb / .kicad_sch (reworked P1 net + routing)
- Regenerate fabrication outputs (gerbers, drill, STEP, DRC: 0 errors, 0 unconnected)
- Re-render top/bottom/perspective with P1 shown, now that it's functional
- README: document short-P1-to-write-protect

Co-Authored-By: Claude Opus 4.8 (1M context) <noreply@anthropic.com>
Connections:
- net +3.3V: now also P1.2
- net GND: no longer P1.2
Changed lines of the file:
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@@
+	)
+	(symbol
+		(lib_id "power:+3.3V")
+		(at 234.95 64.77 180)
+		(unit 1)
+		(exclude_from_sim no)
+		(in_bom yes)
+		(on_board yes)
+		(dnp no)
+		(fields_autoplaced yes)
+		(property "Reference" "#PWR01"
+			(at 234.95 60.96 0)
+			(effects
+				(font
+					(size 1.27 1.27)
+				)
+				(hide yes)
+			)
+		)
+		(property "Value" "+3.3V"
+			(at 234.95 69.85 0)
+			(effects
+				(font
+					(size 1.27 1.27)
+				)
+			)
+		)
+		(property "Footprint" ""
+			(at 234.95 64.77 0)
+			(effects
+				(font
+					(size 1.27 1.27)
+				)
+				(hide yes)
+			)
+		)
+		(property "Datasheet" ""
+			(at 234.95 64.77 0)
+			(effects
+				(font
+					(size 1.27 1.27)
+				)
+				(hide yes)
+			)
+		)
+		(property "Description" "Power symbol creates a global label with name \"+3.3V\""
+			(at 234.95 64.77 0)
+			(effects
+				(font
+					(size 1.27 1.27)
+				)
+				(hide yes)
+			)
+		)
+		(pin "1"
+		)
+		(instances
+			(project "codemyriad-protogon"
+				(path "/fb9bfa6e-c44d-469c-aa90-8ec28bcdf17f"
+					(reference "#PWR01")
+					(unit 1)
+				)
+			)
+		)
 	)
 	(symbol
@@
 					(unit 1)
 				)
-			)
-		)
-	)
-	(symbol
-		(lib_id "power:GND")
-		(at 234.95 64.77 0)
-		(unit 1)
-		(exclude_from_sim no)
-		(in_bom yes)
-		(on_board yes)
-		(dnp no)
-		(fields_autoplaced yes)
-		(property "Reference" "#PWR01"
-			(at 234.95 71.12 0)
-			(effects
-				(font
-					(size 1.27 1.27)
-				)
-				(hide yes)
-			)
-		)
-		(property "Value" "GND"
-			(at 234.95 69.85 0)
-			(effects
-				(font
-					(size 1.27 1.27)
-				)
-			)
-		)
-		(property "Footprint" ""
-			(at 234.95 64.77 0)
-			(effects
-				(font
-					(size 1.27 1.27)
-				)
-				(hide yes)
-			)
-		)
-		(property "Datasheet" ""
-			(at 234.95 64.77 0)
-			(effects
-				(font
-					(size 1.27 1.27)
-				)
-				(hide yes)
-			)
-		)
-		(property "Description" "Power symbol creates a global label with name \"GND\" , ground"
-			(at 234.95 64.77 0)
-			(effects
-				(font
-					(size 1.27 1.27)
-				)
-				(hide yes)
-			)
-		)
-		(pin "1"
-		)
-		(instances
-			(project ""
-				(path "/fb9bfa6e-c44d-469c-aa90-8ec28bcdf17f"
-					(reference "#PWR01")
-					(unit 1)
-				)

Commit message: Fix Qwiic VCC net + dangling label; enable DFM clearance rules
Critical finding from the review: U2 pin 2 (Qwiic VCC) sat on a dead /3V3
net, never joined to +3.3V, so a Qwiic sensor got no power. Fixes:

- PCB: reassign U2 pad 2 from /3V3 to +3.3V (the actual bug). This leaves
  exactly one ratsnest, U2.2 -> P1.2, for the final track (see note).
- Schematic: relabel the dangling "3V3" label to "+3.3V" -> ERC is now
  clean (this was the board's only ERC error).
- Design rules: enable min_copper_edge_clearance (0.25 mm) and
  min_silk_clearance (0.1 mm); the board passes both.

The U2.2 -> +3.3V copper is left for KiCad's interactive router: B.Cu carries
a GND pour and U2.2 is the middle pin of a 1 mm-pitch connector with +3.3V on
the far side, so a clean route needs live DRC and zone refill. One short track.

Co-Authored-By: Claude Opus 4.8 (1M context) <noreply@anthropic.com>
Connections:
- net 3V3 is gone; now on net +3.3V: U2.2
Changed lines of the file:
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@@
 		)
 	)
-	(label "3V3"
+	(label "+3.3V"
 		(at 168.91 132.08 0)
 		(effects
