File: codemyriad-protogon.kicad_sch (KiCad schematic)
At the start: 13 parts, among them J1 Hexpansion-Connector, J2 Conn_02x10_Odd_Even, P1 PZ254V-11-02P, U1 ZD24C64A-XGMT, U2 SM04B-SRSS-TB_(LF)(SN)

Commit message: Route the Qwiic VCC; board is DRC/ERC clean and order-ready
The designer routed the one remaining track (U2 pin 2 → +3.3V), closing the
Qwiic-power bug from the review. Board files are from their KiCad save;
fabrication outputs and renders regenerated to match.

- U2.2 Qwiic VCC now on +3.3V and routed: DRC 0 errors, 0 unconnected
- ERC clean; no orphan nets
- Re-verified vs spec: edge-connector pinout (all 20), EEPROM at 0x50,
  SDA/SCL, 4K7 pull-ups, WP jumper, decoupling, detect→GND
- Regenerate gerbers, drill, STEP, positions, DRC report, renders

Co-Authored-By: Claude Opus 4.8 (1M context) <noreply@anthropic.com>
Connections:
- net 3V3 is gone; now on net +3.3V: U2.2
Changed lines of the file:
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@@
+	(wire
+		(pts
+			(xy 165.1 132.08) (xy 176.53 132.08)
+		)
+		(stroke
+			(width 0)
+			(type default)
+		)
+	)
 	(wire
 		(pts
@@
 	(wire
 		(pts
-			(xy 168.91 132.08) (xy 176.53 132.08)
-		)
-		(stroke
-			(width 0)
-			(type default)
-		)
-	)
-	(wire
-		(pts
 			(xy 186.69 46.99) (xy 195.58 46.99)
 		)
@@
 		(pts
 			(xy 195.58 46.99) (xy 204.47 46.99)
+		)
+		(stroke
+			(width 0)
+			(type default)
+		)
+	)
+	(wire
+		(pts
+			(xy 165.1 132.08) (xy 165.1 128.27)
 		)
 		(stroke
@@
 	(label "HS_G"
 		(at 77.47 80.01 0)
-		(effects
-			(font
-				(size 1.27 1.27)
-			)
-			(justify left bottom)
-		)
-	)
-	(label "3V3"
-		(at 168.91 132.08 0)
 		(effects
 			(font
@@
 					(unit 1)
 				)
+			)
+		)
+	)
+	(symbol
+		(lib_id "power:+3.3V")
+		(at 165.1 128.27 0)
+		(unit 1)
+		(exclude_from_sim no)
+		(in_bom yes)
+		(on_board yes)
+		(dnp no)
+		(fields_autoplaced yes)
+		(property "Reference" "#PWR014"
+			(at 165.1 132.08 0)
+			(effects
+				(font
+					(size 1.27 1.27)
+				)
+				(hide yes)
+			)
+		)
+		(property "Value" "+3.3V"
+			(at 165.1 123.19 0)
+			(effects
+				(font
+					(size 1.27 1.27)
+				)
+			)
+		)
+		(property "Footprint" ""
+			(at 165.1 128.27 0)
+			(effects
+				(font
+					(size 1.27 1.27)
+				)
+				(hide yes)
+			)
+		)
+		(property "Datasheet" ""
+			(at 165.1 128.27 0)
+			(effects
+				(font
+					(size 1.27 1.27)
+				)
+				(hide yes)
+			)
+		)
+		(property "Description" "Power symbol creates a global label with name \"+3.3V\""
+			(at 165.1 128.27 0)
+			(effects
+				(font
+					(size 1.27 1.27)
+				)
+				(hide yes)
+			)
+		)
+		(pin "1"
+		)
+		(instances
+			(project ""
+				(path "/fb9bfa6e-c44d-469c-aa90-8ec28bcdf17f"
+					(reference "#PWR014")
+					(unit 1)
+				)
