File: codemyriad-protogon.kicad_sch (KiCad schematic)
At the start: 13 parts, among them J1 Hexpansion-Connector, J2 Conn_02x10_Odd_Even, P1 PZ254V-11-02P, U1 ZD24C64A-XGMT, U2 SM04B-SRSS-TB_(LF)(SN)

Commit message: Fix missing surface components from rendering
Parts:
- J2, P1: now not fitted
Changed lines of the file:
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@@
 		(in_bom yes)
 		(on_board yes)
-		(dnp no)
+		(dnp yes)
 		(fields_autoplaced yes)
 		(property "Reference" "P1"
@@
 		(in_bom yes)
 		(on_board yes)
-		(dnp no)
+		(dnp yes)
 		(property "Reference" "J2"
 			(at 112.776 53.086 0)
