File: codemyriad-protogon.kicad_pcb (KiCad board)
At the start: 2 copper layers, 54.3 x 36.6 mm, 14 parts, among them J1 Hexpansion-Connector, J2 Conn_02x10_Odd_Even, P1 PZ254V-11-02P, U1 ZD24C64A-XGMT, U2 SM04B-SRSS-TB_(LF)(SN)

Commit message: Rotate text
Other:
- board text removed: "PROTOGON"
