File: codemyriad-protogon.kicad_pcb (KiCad board)
At the start: 2 copper layers, 54.3 x 36.6 mm, 14 parts, among them J1 Hexpansion-Connector, J2 Conn_02x10_Odd_Even, P1 PZ254V-11-02P, U1 ZD24C64A-XGMT, U2 SM04B-SRSS-TB_(LF)(SN)

Commit message: Add 'kongroo' to the top silkscreen
Lowercase, bold, 30° along the top-left chamfer — the front-side twin
of 'protogon' on the bottom face (same anchor, size and slant). Front
silk only: all other gerber layers byte-identical, DRC clean. Fab zip
and renders regenerated.

Co-Authored-By: Claude Fable 5 <noreply@anthropic.com>
Other:
- board text added: "kongroo"
Changed lines of the file:
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@@
+		)
+	)
+	(gr_text "kongroo"
+		(at 105 89.5 30)
+		(layer "F.SilkS")
+		(effects
+			(font
+				(size 0.8 0.8)
+				(thickness 0.16)
+				(bold yes)
+			)
 		)
 	)
